File: wchlink.kicad_pcb (KiCad board)
At the start: 2 copper layers, 13 x 32.5 mm, 25 parts, among them J1 USB_C_Receptacle_USB2.0_16P, J2 Conn_02x04_Odd_Even, SW1 SW_Push, SW2 SW_Push, U1 CH549G, U2 RT9193-33GB

Commit message: 内嵌了3d模型
Parts:
- U1: footprint Package_SO:SOP-16_3.9x9.9mm_P1.27mm -> my_footprint:SOP-16_3.9x9.9mm_P1.27mm
